File: kicad/clock.kicad_pcb (KiCad board)
At the start: 2 copper layers, 137.5 x 91 mm, 60 parts, among them J1 USB_C_Receptacle_PowerOnly_6P, J2 USB_A, J5 Barrel_Jack, SW1 SW_SPDT, SW2 SW_Push, SW3 SW_Push, U1 4511, U10 4060, U11 4013, U12 D1X8K-14BL, U13 D1X8K-14BL, U14 D1X8K-14BL, U15 D1X8K-14BL, U16 D1X8K-14BL, U17 D1X8K-14BL, U18 4081, U2 4511, U3 4511, U4 4511, U5 4511, U6 4511, U7 4518, U8 4518, U9 4518, Y1 32768

Commit message: Add qr code etc
Parts:
- added G001: LOGO, 80_Bus:qr-code, B.Cu at (180.5, 91.5)
Other:
- board text added: "Docs -->>"

Commit message: Update docs
Other:
- board text added: "V1.4"
- board text removed: "V1.2"
Changed lines of the file:
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@@
 	(title_block
 		(title "Logic Clock")
-		(date "2025-11-16")
-		(rev "1.2")
+		(date "2025-11-27")
+		(rev "1.4")
 	)
 	(layers
@@
 		)
 	)
-	(gr_text "V1.2"
+	(gr_text "V1.4"
 		(at 121.5 171.5 0)
 		(layer "F.SilkS")

Commit message: Documentation
Parts:
- added SW4: SW_Push, Button_Switch_THT:SW_PUSH_6mm_H5mm, F.Cu at (238.8, 134.8)
Connections:
- RN6 pad 1: unconnected-(RN6-R1.1-Pad1) -> VDD
- RN6 pad 16: unconnected-(RN6-R1.2-Pad16) -> TEST
- U1 pad 3: VDD -> TEST
- U2 pad 3: VDD -> TEST
- U3 pad 3: VDD -> TEST
- U4 pad 3: VDD -> TEST
- U5 pad 3: VDD -> TEST
- U6 pad 3: VDD -> TEST
Routing:
- net TEST: track 0.00 -> 185.2 mm, vias 0 -> 8
- net GND: track 897.2 -> 908.7 mm
- net VDD: track 639.2 -> 628.3 mm
- net Net-(U6-DA): track 35.9 -> 32.6 mm
- net Net-(RN6-R3.2): track 30.2 -> 28.3 mm, vias 0 -> 1
- net CLOCK: track 192.0 -> 191.4 mm
Other:
- board text added: "TEST"
- board text added: "V1.5"
- board text added: "V1.5 - Add test button"
- board text removed: "V1.4"
