File: kicad/clock.kicad_sch (KiCad schematic)
At the start: 59 parts, among them J1 USB_C_Receptacle_PowerOnly_6P, J2 USB_A, J5 Barrel_Jack, SW1 SW_SPDT, SW2 SW_Push, SW3 SW_Push, U1 4511, U10 4060, U11 4013, U12 D1X8K-14BL, U13 D1X8K-14BL, U14 D1X8K-14BL, U15 D1X8K-14BL, U16 D1X8K-14BL, U17 D1X8K-14BL, U18 4081, U2 4511, U3 4511, U4 4511, U5 4511, U6 4511, U7 4518, U8 4518, U9 4518, Y1 32768

Commit message: Update docs
Other:
- note added: "5161AS - Red 5161AO - Orange (Never found one!) 5161AY - Yellow 5161AG - Olivine 5161AGG - Emerald 5611AB - Blue 5161AW - White SC56-11SYKWA - Bright Yellow"
Changed lines of the file:
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@@
 	(title_block
 		(title "Logic Clock")
-		(date "2025-10-31")
-		(rev "1.0")
+		(date "2025-11-27")
+		(rev "1.4")
 	)
 	(text "Unused Device"
@@
 		)
 	)
+	(text "5161AS  - Red\n5161AO  - Orange (Never found one!)\n5161AY  - Yellow\n5161AG  - Olivine\n5161AGG - Emerald\n5611AB  - Blue\n5161AW  - White\n\nSC56-11SYKWA - Bright Yellow\n\n"
+		(exclude_from_sim no)
+		(at 366.014 85.09 0)
+		(effects
+			(font
+				(size 1.27 1.27)
+				(thickness 0.254)
+				(bold yes)
+			)
+			(justify left)
+		)
+	)

Commit message: Documentation
Parts:
- added SW4: SW_Push, Button_Switch_THT:SW_PUSH_6mm_H5mm, symbol Switch:SW_Push
Connections:
- net GND: now also SW4.2
- net VDD: now also RN6.1 (R1.1); no longer U1.3 (~{LT}), U2.3 (~{LT}), U3.3 (~{LT}), U4.3 (~{LT}), U5.3 (~{LT}), U6.3 (~{LT})
- net TEST: now reaches RN6.16 (R1.2)
- net TEST: now also U1.3 (~{LT}), U2.3 (~{LT}), U3.3 (~{LT}), U4.3 (~{LT}), U5.3 (~{LT}), U6.3 (~{LT}), SW4.1
- no-connect marks 25 -> 23
